File: KiCad/file5BC7F38B.sch (KiCad schematic (older format))
At the start: 78 parts, among them J301 DB9_Female, J302 Conn_01x06, J303 DB9_Male, J304 Conn_01x10, J305 Conn_01x02, J306 Conn_01x02, J307 Conn_01x02, J308 Conn_01x02, P301 ISP/PDI, P302 Thru, P304 Header, Q301 PN2222A, SW301 SPST, U301 DS3231, U302 AVR128DA48, U303 LD2985BM33R, U304 SI5351A, U305 74HC1G08, U306 LT1763CS8-5, U307 TPS22810DBVT, U308 LD2985BM33R, X301 25.MHZ TCXO

Commit message: Latest Gerbers
Gerbers with minor updates to silkscreen and D101, D301 footprints
Parts:
- D301: footprint TO_SOT_Packages_SMD:SOT-363-0.65 -> TO_SOT_Packages_SMD:SOT-363-0.65_MBD54
- D304, D305: footprint Resistors_SMD:R_0805 -> Diodes_SMD:D_0805
Changed lines of the file:
@@
 F 0 "D305" H 10350 5250 50  0000 C CNN
 F 1 "RED" H 10400 5050 50  0000 C CNN
-F 2 "Resistors_SMD:R_0805" H 10350 5150 50  0001 C CNN
+F 2 "Diodes_SMD:D_0805" H 10350 5150 50  0001 C CNN
 F 3 "" H 10350 5150 50  0001 C CNN
 F 4 "732-4984-1-ND " H 10350 5150 50  0001 C CNN "Digi-Key Part No."
@@
 F 0 "D301" H 2900 8350 50  0000 C CNN
 F 1 "MBD54" H 2925 8725 50  0001 C CNN
-F 2 "TO_SOT_Packages_SMD:SOT-363-0.65" H 2900 8450 50  0001 C CNN
+F 2 "TO_SOT_Packages_SMD:SOT-363-0.65_MBD54" H 2900 8450 50  0001 C CNN
 F 3 "" H 2900 8450 50  0001 C CNN
 F 4 "MBD54DWT1GOSCT-ND" H 2900 8450 50  0001 C CNN "Digi-Key Part No."
@@
 F 0 "D304" H 11150 5200 50  0000 C CNN
 F 1 "GREEN" H 11200 5400 50  0000 C CNN
-F 2 "Resistors_SMD:R_0805" H 11150 5300 50  0001 C CNN
+F 2 "Diodes_SMD:D_0805" H 11150 5300 50  0001 C CNN
 F 3 "" H 11150 5300 50  0001 C CNN
 F 4 "732-4983-1-ND" H 11150 5300 50  0001 C CNN "Digi-Key Part No."
