File: KiCad/file591BC95F.sch (KiCad schematic (older format))
At the start: 39 parts, among them J203 V4, P201 AUX BATTERY, P202 To Power Supply Board, P203 AUX BATTERY, U201 DAC081C085, U202 OPA171, U203 LTC3600

Commit message: Changes for FlexFox80
Wholesale changes for new project.
Parts:
- J203: symbol ARDF-2-Band-MiniTx-rescue:CONN_01X01 -> FlexFox80-rescue:CONN_01X01-ARDF-2-Band-MiniTx-rescue
- L201, L202: symbol ARDF-2-Band-MiniTx-rescue:INDUCTOR_SMALL -> FlexFox80-rescue:INDUCTOR_SMALL-ARDF-2-Band-MiniTx-rescue
- P201, P203: symbol ARDF-2-Band-MiniTx-rescue:CONN_01X02 -> FlexFox80-rescue:CONN_01X02-ARDF-2-Band-MiniTx-rescue
- P202: symbol ARDF-2-Band-MiniTx-rescue:CONN_02X06 -> FlexFox80-rescue:CONN_02X06-ARDF-2-Band-MiniTx-rescue
- U201: symbol ARDF-2-Band-MiniTx-rescue:DAC081C085 -> FlexFox80-rescue:DAC081C085-ARDF-2-Band-MiniTx-rescue
- U202: symbol ARDF-2-Band-MiniTx-rescue:OPA171 -> FlexFox80-rescue:OPA171-ARDF-2-Band-MiniTx-rescue
- U203: symbol ARDF-2-Band-MiniTx-rescue:LTC3600 -> FlexFox80-rescue:LTC3600-ARDF-2-Band-MiniTx-rescue
- W201: symbol ARDF-2-Band-MiniTx-rescue:TEST_1P -> FlexFox80-rescue:TEST_1P-ARDF-2-Band-MiniTx-rescue
- W202, W203, W204, W205: symbol ARDF-2-Band-MiniTx-rescue:TEST_SCOPE -> FlexFox80-rescue:TEST_SCOPE-ARDF-2-Band-MiniTx-rescue
Connections:
- wire segments 96 -> 128
Other:
- note added: "PCB: Flex Fox 80 ARDF Transmitter (p. 2/3)"
- note removed: "PCB: Dual-Band Transmitter (p. 2/3)"

Commit message: Updates to Schematic
Updates to Schematic
Parts:
- removed D201: B530, Diodes_SMD:DO-214AB_Handsoldering, symbol Device:D_Schottky
- removed P201: AUX BATTERY, Oddities:Dummy_Empty_2, symbol FlexFox80-rescue:CONN_01X02-ARDF-2-Band-MiniTx-rescue
- removed P202: To Power Supply Board, Pin_Headers:Pin_Header_Straight_2x06, symbol FlexFox80-rescue:CONN_02X06-ARDF-2-Band-MiniTx-rescue
- removed W201: Vin, Measurement_Points:Measurement_Point_Round-SMD-Pad_Small, symbol FlexFox80-rescue:TEST_1P-ARDF-2-Band-MiniTx-rescue
- removed W202: Vbat, Measurement_Points:Measurement_Point_ScopeProbe_Round-SMD-2sides-Pad_Small, symbol FlexFox80-rescue:TEST_SCOPE-ARDF-2-Band-MiniTx-rescue
- removed W203: +12V, Measurement_Points:Measurement_Point_ScopeProbe_Round-SMD-2sides-Pad_Small, symbol FlexFox80-rescue:TEST_SCOPE-ARDF-2-Band-MiniTx-rescue
- added C?: 47uF, Capacitors_SMD:C_1210_HandSoldering, symbol Device:C_Small
- added C?: 10uF, Capacitors_SMD:C_1210_HandSoldering, symbol Device:C_Small
- added C?: 100nF, Capacitors_SMD:C_0805_HandSoldering, symbol Device:C_Small
- added C?: 1uF, Capacitors_SMD:C_0805_HandSoldering, symbol Device:C_Small
- added C? (x2): 150uF low ESR, Capacitors_SMD:C_2917_7343_Metric_HandSoldering, symbol Device:CP1_Small
- added C?: 10nF, Capacitors_SMD:C_0805_HandSoldering, symbol Device:C_Small
- added D? (x2): B530, Diodes_SMD:DO-214AB_Handsoldering, symbol Device:D_Schottky_ALT
- added L?: 6.8uH, Inductors:CDR7D28MN, symbol FlexFox80-rescue:INDUCTOR_SMALL-ARDF-2-Band-MiniTx-rescue
- added P?: Power Pole, symbol FlexFox80-rescue:CONN_01X02-ARDF-2-Band-MiniTx-rescue
- added Q? (x2): DMP4025LSD, SO-8, symbol Transistor_FET:DMP4025LSD
- added Q?: AO4576, SO-8, symbol Transistor_FET:SI4884BDY
- added Q?: MUN5211, SO-8, symbol Transistor_Array:MUN5211DW1T1G
- added R?: 100k, Resistors_SMD:R_0805_HandSoldering, symbol Device:R
- added R? (x3): 10k, Resistors_SMD:R_0805_HandSoldering, symbol Device:R
- added R?: 1.1k, Resistors_SMD:R_0805_HandSoldering, symbol Device:R
- added R?: 0.01 0.5W, Resistors_SMD:R_0805_HandSoldering, symbol Device:R
- added U?: MIC2196, symbol Power_Management:MIC2196
- P203: value AUX BATTERY -> Power Pole; footprint Sockets:Phoenix_3.81mm_2pos -> (none); Description (none) -> TH; Link <a href=\"https://www.digikey.com/products/en?keywords=277-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 -> <a href=\"https://www.digikey.com/products/en?keywords=2243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; Manufacturer (none) -> TH; Manufacturer PN (none) -> TH; Part No. 277-1206-ND -> 2243-ASMPP30-1X2-RK-ND
- R213: value 12.4k -> 10k
Connections:
- net labels added: BOOST_ENABLE, EXTERNAL_3.2V-12V_SUPPLY
- net labels removed: AUX_BAT_DIRECT, MAIN_PWR_ENABLE, VBAT_UNINTERRUPTED
- wire segments 128 -> 162
Other:
- note added: "+11.5V => 15k & 1.8k\n+12.5V => 10k & 1.1k\n+12.8V => 14k & 1.5k\n+13.6V => 15k & 1.5k"
- note added: "Close to pin 6"
- note added: "External Battery\nConnector"
- note added: "High-Efficiency Boost Power Regulator"
- note added: "High-Efficiency Variable Buck Power Regulator"
- note removed: "Auxiliary Battery\nConnector"
- note removed: "High-Efficiency Buck Power Regulator"
- note removed: "Power Supply Board\nConnector"
- note removed: "Vbat <= 4.5V"
- moved on the sheet: C202, C204, P203, R201, R202, R205, R213

Commit message: Design Updates
Specifying components
Parts:
- removed C?: 47uF, Capacitors_SMD:C_1210_HandSoldering, symbol Device:C_Small
- removed C?: 10uF, Capacitors_SMD:C_1210_HandSoldering, symbol Device:C_Small
- removed C?: 1uF, Capacitors_SMD:C_0805_HandSoldering, symbol Device:C_Small
- removed C?: 150uF low ESR, Capacitors_SMD:C_2917_7343_Metric_HandSoldering, symbol Device:CP1_Small
- removed D?: B530, Diodes_SMD:DO-214AB_Handsoldering, symbol Device:D_Schottky_ALT
- removed Q?: DMP4025LSD, SO-8, symbol Transistor_FET:DMP4025LSD
- removed Q?: MUN5211, SO-8, symbol Transistor_Array:MUN5211DW1T1G
- removed R? (x2): 10k, Resistors_SMD:R_0805_HandSoldering, symbol Device:R
- added C209: 150uF low ESR, Capacitors_SMD:C_2917_7343_Metric_HandSoldering, symbol Device:CP1_Small
- added C216: 10uF, Capacitors_SMD:C_0805, symbol Device:C_Small
- added C217: 47uF low ESR, Capacitors_SMD:C_2917_7343_Metric_HandSoldering, symbol Device:CP1_Small
- added C219: 1uF, Capacitors_SMD:C_0805, symbol Device:C_Small
- added D201: B530, Diodes_SMD:DO-214AB, symbol Device:D_Schottky_ALT
- added Q201: MUN5213DW1, TO_SOT_Packages_SMD:SOT-363-0.65, symbol Transistor_BJT:MUN5213DW1
- added unit 2 of Q202
- added R215, R216: 10k, Resistors_SMD:R_0805, symbol Device:R
- C201, C203, C205: footprint Capacitors_SMD:C_0805_HandSoldering -> Capacitors_SMD:C_0805; Description (none) -> CAP CER 10UF 25V X5R 0805; Digi-Key Part No. (none) -> 490-5523-1-ND; Manufacturer (none) -> Murata Electronics; Manufacturer PN (none) -> GRM21BR61E106KA73L; Part No. 490-5523-1-ND -> (none)
- C202, C204, C211, C212: footprint Capacitors_SMD:C_0805_HandSoldering -> Capacitors_SMD:C_0805; Description (none) -> CAP CER 0.1UF 50V X7R 0805; Digi-Key Part No. (none) -> 478-1395-1-ND; Manufacturer (none) -> AVX Corporation; Manufacturer PN (none) -> 08055C104KAT2A; Part No. 478-1395-1-ND -> (none)
- C206: renamed from C?; footprint Capacitors_SMD:C_0805_HandSoldering -> Capacitors_SMD:C_0805; Description (none) -> CAP CER 0.1UF 50V X7R 0805; Digi-Key Part No. (none) -> 478-1395-1-ND; Manufacturer (none) -> AVX Corporation; Manufacturer PN (none) -> 08055C104KAT2A; Part No. 478-1395-1-ND -> (none)
- C207: footprint Capacitors_SMD:C_0805_HandSoldering -> Capacitors_SMD:C_0805; Description (none) -> CAP CER 270PF 50V C0G/NP0 0805; Digi-Key Part No. (none) -> 1276-2624-1-ND; Manufacturer (none) -> Samsung Electro-Mechanics; Manufacturer PN (none) -> CL21C271GBANNNC; Part No. 1276-2624-1-ND -> (none)
- C208: footprint Capacitors_SMD:C_0805_HandSoldering -> Capacitors_SMD:C_0805; Description (none) -> CAP CER 10PF 200V C0G/NP0 0805; Digi-Key Part No. (none) -> 478-10457-1-ND; Manufacturer (none) -> AVX Corporation; Manufacturer PN (none) -> 08052U100FAT2A; Part No. 478-10457-1-ND -> (none)
- C210: footprint Capacitors_SMD:C_1210_HandSoldering -> Capacitors_SMD:C_1210; Description (none) -> CAP CER 22UF 25V X5R 1210; Digi-Key Part No. (none) -> 1276-3373-1-ND; Manufacturer (none) -> Samsung Electro-Mechanics; Manufacturer PN (none) -> CL32A226MAJNNNE; Part No. 1276-3373-1-ND -> (none)
- C213: footprint Capacitors_SMD:C_0805_HandSoldering -> Capacitors_SMD:C_0805; Description (none) -> CAP CER 1UF 16V X7R 0805; Digi-Key Part No. (none) -> 311-1365-1-ND; Manufacturer (none) -> Yageo; Manufacturer PN (none) -> CC0805KKX7R7BB105; Part No. 311-1365-1-ND -> (none)
- C214: Description (none) -> CAP TANT 47UF 10% 20V 2917; Digi-Key Part No. (none) -> 399-3904-1-ND; Link <a href=\"https://www.digikey.com/products/en?keywords=399-3885-1-ND\">Link</a> -> <a href=\"https://www.digikey.com/products/en?keywords=399-3904-1-ND\">Link</a>; Manufacturer (none) -> KEMET; Manufacturer PN (none) -> T495X476K020ATE150; Part No. 399-3885-1-ND -> (none)
- C215: renamed from C?; Description (none) -> CAP TANT 150UF 10% 20V 2917; Digi-Key Part No. (none) -> 478-5253-1-ND; Link <a href=\"https://www.digikey.com/products/en?keywords=399-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 -> <a href=\"https://www.digikey.com/products/en?keywords=478-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; Manufacturer (none) -> AVX Corporation; Manufacturer PN (none) -> TPME157K020R0035; Part No. 399-3885-1-ND -> (none)
- C218: renamed from C?; footprint Capacitors_SMD:C_0805_HandSoldering -> Capacitors_SMD:C_0805; Description (none) -> CAP CER 10000PF 50V NP0 0805; Digi-Key Part No. (none) -> 478-10068-1-ND; Link <a href=\"https://www.digikey.com/products/en?keywords=490-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 -> <a href=\"https://www.digikey.com/products/en?keywords=478-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; Manufacturer (none) -> AVX Corporation; Manufacturer PN (none) -> 08055A103JAT2A; Part No. 490-5523-1-ND -> (none)
- D202: renamed from D?; footprint Diodes_SMD:DO-214AB_Handsoldering -> Diodes_SMD:DO-214AB; Digi-Key Part No. (none) -> B530C-FDICT-ND; Part No. B530C-FDICT-ND -> (none)
- J203, W204, W205: Digi-Key Part No. (none) -> np; Part No. np -> (none)
- L201: footprint Resistors_SMD:R_0805_HandSoldering -> Resistors_SMD:R_0805; Description (none) -> FIXED IND 10UH 100MA 390 MOHM; Digi-Key Part No. (none) -> 490-6682-1-ND; Link <a href=\"https://www.digikey.com/products/en?keywords=445-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 -> <a href=\"https://www.digikey.com/products/en?keywords=490-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; Manufacturer (none) -> Murata Electronics; Manufacturer PN (none) -> LQM21FN100M80L; Part No. 445-6396-1-ND -> (none)
- L202: Description (none) -> FIXED IND 6.8UH 2.75A 46.3 MOHM; Digi-Key Part No. (none) -> 308-1328-1-ND; Manufacturer (none) -> Sumida America Components Inc.; Manufacturer PN (none) -> CDR7D28MNNP-6R8NC; Part No. 308-1328-1-ND -> (none)
- L203: renamed from L?; Description (none) -> FIXED IND 6.8UH 2.75A 46.3 MOHM; Digi-Key Part No. (none) -> 308-1328-1-ND; Manufacturer (none) -> Sumida America Components Inc.; Manufacturer PN (none) -> CDR7D28MNNP-6R8NC; Part No. 308-1328-1-ND -> (none)
- P201: renamed from P?; Digi-Key Part No. (none) -> 2243-ASMPP30-1X2-RK-ND; Part No. 2243-ASMPP30-1X2-RK-ND -> (none)
- P203: Digi-Key Part No. (none) -> 2243-ASMPP30-1X2-RK-ND; Part No. 2243-ASMPP30-1X2-RK-ND -> (none)
- Q202: renamed from Q?; footprint SO-8 -> Housings_SOIC:SOIC-8_3.9x4.9mm_Pitch1.27mm; Description (none) -> MOSFET 2P-CH 40V 6.9A 8SO; Digi-Key Part No. (none) -> DMP4025LSD-13DICT-ND; Link (none) -> <a href=\"https://www.digikey.com/products/en?keywords=DMP4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; Manufacturer (none) -> Diodes Incorporated; Manufacturer PN (none) -> DMP4025LSD-13
- Q203: renamed from Q?; value AO4576 -> RJK0354DSP; footprint SO-8 -> Housings_SOIC:SOIC-8_3.9x4.9mm_Pitch1.27mm; Description (none) -> MOSFET N-CH 30V 16A 8SOP; Digi-Key Part No. (none) -> RJK0354DSP-00#J0CT-ND; Link (none) -> <a href=\"https://www.digikey.com/products/en?keywords=RJK0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; Manufacturer (none) -> Renesas Electronics America Inc; Manufacturer PN (none) -> RJK0354DSP-00#J0
- R201, R205, R212: footprint Resistors_SMD:R_0805_HandSoldering -> Resistors_SMD:R_0805; Description (none) -> RES SMD 162K OHM 1% 1/8W 0805; Digi-Key Part No. (none) -> 311-162KCRCT-ND; Manufacturer (none) -> Yageo; Manufacturer PN (none) -> RC0805FR-07162KL; Part No. 311-162KCRCT-ND -> (none)
- R202: Description (none) -> RES SMD 49.9K OHM 0.1% 1/8W 0805; Digi-Key Part No. (none) -> YAG4990CT-ND; Link <a href=\"https://www.digikey.com/products/en?keywords=RMCF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 -> <a href=\"https://www.digikey.com/products/en?keywords=YAG4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; Manufacturer (none) -> Yageo; Manufacturer PN (none) -> RT0805BRE0749K9L; Part No. RMCF0805FT49K9CT-ND -> (none)
- R203, R208: footprint Resistors_SMD:R_0805_HandSoldering -> Resistors_SMD:R_0805; Description (none) -> RES SMD 27K OHM 1% 1/8W 0805; Digi-Key Part No. (none) -> 311-27.0KCRCT-ND; Manufacturer (none) -> Yageo; Manufacturer PN (none) -> RC0805FR-0727KL; Part No. 311-27.0KCRCT-ND -> (none)
- R204: footprint Resistors_SMD:R_0805_HandSoldering -> Resistors_SMD:R_0805; Description (none) -> RES SMD 536K OHM 1% 1/8W 0805; Digi-Key Part No. (none) -> 311-536KCRCT-ND; Manufacturer (none) -> Yageo; Manufacturer PN (none) -> RC0805FR-07536KL; Part No. 311-536KCRCT-ND -> (none)
- R206: footprint Resistors_SMD:R_0805_HandSoldering -> Resistors_SMD:R_0805; Description (none) -> RES 46.4K OHM 1% 1/8W 0805; Digi-Key Part No. (none) -> RMCF0805FT46K4CT-ND; Manufacturer (none) -> Stackpole Electronics Inc; Manufacturer PN (none) -> RMCF0805FT46K4; Part No. RMCF0805FT46K4CT-ND -> (none)
- R207, R210: footprint Resistors_SMD:R_0805_HandSoldering -> Resistors_SMD:R_0805; Description (none) -> RES SMD 100K OHM 1% 1/8W 0805; Digi-Key Part No. (none) -> 311-100KCRCT-ND; Manufacturer (none) -> Yageo; Manufacturer PN (none) -> RC0805FR-07100KL; Part No. 311-100KCRCT-ND -> (none)
- R209: renamed from R?; footprint Resistors_SMD:R_0805_HandSoldering -> Resistors_SMD:R_0805; Description (none) -> RES SMD 100K OHM 1% 1/8W 0805; Digi-Key Part No. (none) -> 311-100KCRCT-ND; Manufacturer (none) -> Yageo; Manufacturer PN (none) -> RC0805FR-07100KL; Part No. 311-100KCRCT-ND -> (none)
- R211: value 12.4k -> 10k; footprint Resistors_SMD:R_0805_HandSoldering -> Resistors_SMD:R_0805; Description (none) -> RES SMD 10K OHM 1% 1/8W 0805; Digi-Key Part No. (none) -> 311-10KLGCT-ND; Link <a href=\"https://www.digikey.com/products/en?keywords=P12.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 -> <a href=\"https://www.digikey.com/products/en?keywords=311-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; Manufacturer (none) -> Yageo; Manufacturer PN (none) -> AC0805FR-0710KL; Part No. P12.4KCCT-ND -> (none)
- R213: footprint Resistors_SMD:R_0805_HandSoldering -> Resistors_SMD:R_0805; Description (none) -> RES SMD 10K OHM 1% 1/8W 0805; Digi-Key Part No. (none) -> 311-10KLGCT-ND; Link <a href=\"https://www.digikey.com/products/en?keywords=P12.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 -> <a href=\"https://www.digikey.com/products/en?keywords=311-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; Manufacturer (none) -> Yageo; Manufacturer PN (none) -> AC0805FR-0710KL; Part No. P12.4KCCT-ND -> (none)
- R214: renamed from R?; footprint Resistors_SMD:R_0805_HandSoldering -> Resistors_SMD:R_0805; Description (none) -> RES SMD 10K OHM 1% 1/8W 0805; Digi-Key Part No. (none) -> 311-10.0KCRCT-ND; Link <a href=\"https://www.digikey.com/products/en?keywords=311-27.0KCRCT-ND\">Link</a> -> <a href=\"https://www.digikey.com/products/en?keywords=311-10.0KCRCT-ND\">Link</a>; Manufacturer (none) -> Yageo; Manufacturer PN (none) -> RC0805FR-0710KL; Part No. 311-27.0KCRCT-ND -> (none)
- R217: renamed from R?; footprint Resistors_SMD:R_0805_HandSoldering -> Resistors_SMD:R_0805; Description (none) -> RES SMD 1.1K OHM 1% 1/8W 0805; Digi-Key Part No. (none) -> 311-1.10KCRCT-ND; Link <a href=\"https://www.digikey.com/products/en?keywords=311-27.0KCRCT-ND\">Link</a> -> <a href=\"https://www.digikey.com/products/en?keywords=311-1.10KCRCT-ND\">Link</a>; Manufacturer (none) -> Yageo; Manufacturer PN (none) -> RC0805FR-071K1L; Part No. 311-27.0KCRCT-ND -> (none)
- R218: renamed from R?; footprint Resistors_SMD:R_0805_HandSoldering -> Resistors_SMD:R_0805; Description (none) -> RES 0.01 OHM 1% 1/2W 0805; Digi-Key Part No. (none) -> 408-1544-1-ND; Link <a href=\"https://www.digikey.com/products/en?keywords=311-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 -> <a href=\"https://www.digikey.com/products/en?keywords=408-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; Manufacturer (none) -> Susumu; Manufacturer PN (none) -> KRL1220E-M-R010-F-T5; Part No. 311-27.0KCRCT-ND -> (none)
- U201: footprint SMD_Packages:SSOP-8_Handsolder -> Housings_SSOP:MSOP-8_3x3mm_Pitch0.65mm; Description (none) -> IC DAC 8BIT V-OUT 8VSSOP; Digi-Key Part No. (none) -> DAC081C085CIMM/NOPBCT-ND; Manufacturer (none) -> Texas Instruments; Manufacturer PN (none) -> DAC081C085CIMM/NOPB; Part No. DAC081C085CIMM/NOPBCT-ND -> (none)
- U202: footprint TO_SOT_Packages_SMD:SOT-23-5_Handsolder -> TO_SOT_Packages_SMD:SOT-23-5_MCP; Description (none) -> IC OPAMP GP 1 CIRCUIT SOT23-5; Digi-Key Part No. (none) -> 296-37698-1-ND; Manufacturer (none) -> Texas Instruments; Manufacturer PN (none) -> OPA171AIDBVR; Part No. 296-37698-1-ND -> (none)
- U203: footprint SMD_Packages:SSOP-12_Pad_Handsolder -> Housings_SSOP:SSOP-12_Pad; Description (none) -> IC REG BUCK PROG 1.5A 12MSOP; Digi-Key Part No. (none) -> LTC3600EMSE#PBF-ND; Manufacturer (none) -> Analog Devices Inc.; Manufacturer PN (none) -> LTC3600EMSE#PBF; Part No. LTC3600EMSE#PBF-ND -> (none)
- U204: renamed from U?; footprint (none) -> Housings_SOIC:SOIC-8_3.9x4.9mm_Pitch1.27mm; Description (none) -> IC REG CTRLR BOOST 8SOIC; Digi-Key Part No. (none) -> MIC2196YM-CT-ND; Link (none) -> <a href=\"https://www.digikey.com/products/en?keywords=MIC2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; Manufacturer (none) -> Microchip Technology; Manufacturer PN (none) -> MIC2196YM-TR
Connections:
- wire segments 162 -> 163

Commit message: Design Updates
Defining parts and footprints
Parts:
- R214: Digi-Key Part No. 311-10.0KCRCT-ND -> 311-10KLGCT-ND; Link <a href=\"https://www.digikey.com/products/en?keywords=311-10.0KCRCT-ND\">Link</a> -> <a href=\"https://www.digikey.com/products/en?keywords=311-10KLGCT-ND\">Link</a>; Manufacturer PN RC0805FR-0710KL -> AC0805FR-0710KL
Changed lines of the file:
@@
 F 2 "Resistors_SMD:R_0805" V 2080 6200 50  0001 C CNN
 F 3 "" H 2150 6200 50  0000 C CNN
-F 4 "311-10.0KCRCT-ND" H 2150 6200 50  0001 C CNN "Digi-Key Part No."
-F 5 "<a href=\"https://www.digikey.com/products/en?keywords=311-10.0KCRCT-ND\">Link</a>" H 2150 6200 60  0001 C CNN "Link"
+F 4 "311-10KLGCT-ND" H 2150 6200 50  0001 C CNN "Digi-Key Part No."
+F 5 "<a href=\"https://www.digikey.com/products/en?keywords=311-10KLGCT-ND\">Link</a>" H 2150 6200 60  0001 C CNN "Link"
 F 6 "Yageo" H 2150 6200 50  0001 C CNN "Manufacturer"
-F 7 "RC0805FR-0710KL" H 2150 6200 50  0001 C CNN "Manufacturer PN"
+F 7 "AC0805FR-0710KL" H 2150 6200 50  0001 C CNN "Manufacturer PN"
 F 8 "RES SMD 10K OHM 1% 1/8W 0805" H 2150 6200 50  0001 C CNN "Description"
 	1    2150 6200

Commit message: Design Updates
Updating schematic parts
Parts:
- C209, C214, C215, C217: footprint Capacitors_SMD:C_2917_7343_Metric_HandSoldering -> Capacitors_SMD:C_2917
- R202: footprint Resistors_SMD:R_0805_HandSoldering -> Resistors_SMD:R_0805
Connections:
- net labels added: MAIN_PWR_ENABLE
- net labels removed: BOOST_ENABLE
Changed lines of the file:
@@
 F 0 "C214" H 8900 2850 50  0000 L CNN
 F 1 "47uF low ESR" H 9350 2850 50  0000 L CNN
-F 2 "Capacitors_SMD:C_2917_7343_Metric_HandSoldering" H 9200 2850 50  0001 C CNN
+F 2 "Capacitors_SMD:C_2917" H 9200 2850 50  0001 C CNN
 F 3 "" H 9200 2850 50  0001 C CNN
 F 4 "399-3904-1-ND" H 9200 2850 50  0001 C CNN "Digi-Key Part No."
@@
 F 0 "C215" V 2000 4850 50  0000 L CNN
 F 1 "150uF low ESR" V 2100 4550 50  0000 L CNN
-F 2 "Capacitors_SMD:C_2917_7343_Metric_HandSoldering" H 1850 4950 50  0001 C CNN
+F 2 "Capacitors_SMD:C_2917" H 1850 4950 50  0001 C CNN
 F 3 "" H 1850 4950 50  0001 C CNN
 F 4 "478-5253-1-ND" H 1850 4950 50  0001 C CNN "Digi-Key Part No."
@@
 F 0 "R202" V 4530 4750 50  0000 C CNN
 F 1 "49.9k" V 4450 4750 50  0000 C CNN
-F 2 "Resistors_SMD:R_0805_HandSoldering" V 4380 4750 50  0001 C CNN
+F 2 "Resistors_SMD:R_0805" V 4380 4750 50  0001 C CNN
 F 3 "" H 4450 4750 50  0001 C CNN
 F 4 "YAG4990CT-ND" H 4450 4750 50  0001 C CNN "Digi-Key Part No."
@@
 	4250 4500 4250 4750
 Text GLabel 4700 6150 2    39   Input ~ 0
-BOOST_ENABLE
+MAIN_PWR_ENABLE
 Wire Wire Line
 	4700 6150 4650 6150
@@
 +11.5V => 15k & 1.8k\n+12.5V => 10k & 1.1k\n+12.8V => 14k & 1.5k\n+13.6V => 15k & 1.5k
 Text GLabel 2700 3850 0    39   Input ~ 0
-BOOST_ENABLE
+MAIN_PWR_ENABLE
 $Comp
 L Device:D_Schottky_ALT D202
@@
 F 0 "C209" V 1600 4650 50  0000 L CNN
 F 1 "150uF low ESR" V 1700 4350 50  0000 L CNN
-F 2 "Capacitors_SMD:C_2917_7343_Metric_HandSoldering" H 1850 4750 50  0001 C CNN
+F 2 "Capacitors_SMD:C_2917" H 1850 4750 50  0001 C CNN
 F 3 "" H 1850 4750 50  0001 C CNN
 F 4 "478-5253-1-ND" H 1850 4750 50  0001 C CNN "Digi-Key Part No."
@@
 F 0 "C217" V 4200 5850 50  0000 L CNN
 F 1 "47uF low ESR" V 4500 5550 50  0000 L CNN
-F 2 "Capacitors_SMD:C_2917_7343_Metric_HandSoldering" H 4350 5950 50  0001 C CNN
+F 2 "Capacitors_SMD:C_2917" H 4350 5950 50  0001 C CNN
 F 3 "" H 4350 5950 50  0001 C CNN
 F 4 "399-3904-1-ND" H 4350 5950 50  0001 C CNN "Digi-Key Part No."

Commit message: Design Updates
Updated schematics parts descriptions
Parts:
- L201: symbol FlexFox80-rescue:INDUCTOR_SMALL-ARDF-2-Band-MiniTx-rescue -> Device:INDUCTOR_SMALL
- P201: footprint (none) -> Oddities:Dummy_Empty_2
- P203: footprint (none) -> Connect:PowerPole-ASMPP30-1x2
- U201: symbol FlexFox80-rescue:DAC081C085-ARDF-2-Band-MiniTx-rescue -> Analog_DAC:DAC081C085
- U202: symbol FlexFox80-rescue:OPA171-ARDF-2-Band-MiniTx-rescue -> Amplifier_Operational:OPA171
- U203: symbol FlexFox80-rescue:LTC3600-ARDF-2-Band-MiniTx-rescue -> Regulator_Switching:LTC3600
- W204: symbol FlexFox80-rescue:TEST_SCOPE-ARDF-2-Band-MiniTx-rescue -> special:TEST_SCOPE
- W205: symbol FlexFox80-rescue:TEST_SCOPE-ARDF-2-Band-MiniTx-rescue -> special:TEST_SCOPE; Manufacturer (none) -> np
Changed lines of the file:
@@
 $EndDescr
 $Comp
-L FlexFox80-rescue:LTC3600-ARDF-2-Band-MiniTx-rescue U203
+L Regulator_Switching:LTC3600 U203
 U 1 1 58B77FB4
 P 7550 2500
@@
 $EndComp
 $Comp
-L FlexFox80-rescue:DAC081C085-ARDF-2-Band-MiniTx-rescue U201
+L Analog_DAC:DAC081C085 U201
 U 1 1 58B84991
 P 3600 2250
@@
 High-Efficiency Variable Buck Power Regulator
 $Comp
-L FlexFox80-rescue:OPA171-ARDF-2-Band-MiniTx-rescue U202
+L Amplifier_Operational:OPA171 U202
 U 1 1 59D417D4
 P 6000 2200
+AR Path="/59D417D4" Ref="U202"  Part="1"
+AR Path="/591BC960/59D417D4" Ref="U202"  Part="1"
 F 0 "U202" H 6000 2450 61  0000 L CNB
 F 1 "OPA171" H 6000 2350 61  0000 L CNB
@@
 F 0 "P203" H 6000 5250 50  0000 C CNN
 F 1 "Power Pole" V 6150 5100 50  0001 C CNN
-F 2 "" H 6000 5100 50  0001 C CNN
+F 2 "Connect:PowerPole-ASMPP30-1x2" H 6000 5100 50  0001 C CNN
 F 3 "" H 6000 5100 50  0001 C CNN
 F 4 "2243-ASMPP30-1X2-RK-ND" H 6000 5100 50  0001 C CNN "Digi-Key Part No."
@@
 	3800 1350 3800 1400
 $Comp
-L FlexFox80-rescue:INDUCTOR_SMALL-ARDF-2-Band-MiniTx-rescue L201
+L Device:INDUCTOR_SMALL L201
 U 1 1 5BF17B46
 P 4350 1650
@@
 NoConn ~ 6500 5150
 $Comp
-L FlexFox80-rescue:TEST_SCOPE-ARDF-2-Band-MiniTx-rescue W204
+L special:TEST_SCOPE W204
 U 1 1 5C0F212A
 P 9400 1500
@@
 $EndComp
 $Comp
-L FlexFox80-rescue:TEST_SCOPE-ARDF-2-Band-MiniTx-rescue W205
+L special:TEST_SCOPE W205
 U 1 1 5F84AD75
 P 4800 2250
@@
 F 4 "np" H 4800 2250 50  0001 C CNN "Digi-Key Part No."
 F 5 "np" H 4800 2250 60  0001 C CNN "Link"
+F 6 "np" H 4800 2250 50  0001 C CNN "Manufacturer"
 	1    4800 2250
 	-1   0    0    1
@@
 F 0 "P201" H 6300 5250 50  0000 C CNN
 F 1 "Power Pole" V 6450 5100 50  0000 C CNN
-F 2 "" H 6300 5100 50  0001 C CNN
+F 2 "Oddities:Dummy_Empty_2" H 6300 5100 50  0001 C CNN
 F 3 "" H 6300 5100 50  0001 C CNN
 F 4 "2243-ASMPP30-1X2-RK-ND" H 6300 5100 50  0001 C CNN "Digi-Key Part No."

Commit message: PCB Updates
o Started PCB layout
Parts:
- P203: symbol FlexFox80-rescue:CONN_01X02-ARDF-2-Band-MiniTx-rescue -> Connector:PowerPole_1x2_pin
Connections:
- net EXTERNAL_3.2V-12V_SUPPLY renamed EXTERNAL_3.6V-15V_SUPPLY
- new net GNDD: P203.E
Changed lines of the file:
@@
 $EndComp
 $Comp
-L FlexFox80-rescue:CONN_01X02-ARDF-2-Band-MiniTx-rescue P203
+L Connector:PowerPole_1x2_pin P203
 U 1 1 59FCFE1A
 P 6000 5100
@@
 $EndComp
 Text GLabel 4250 5450 2    39   Output ~ 0
-EXTERNAL_3.2V-12V_SUPPLY
+EXTERNAL_3.6V-15V_SUPPLY
 Wire Wire Line
 	4250 5450 4100 5450
@@
 Wire Wire Line
 	3500 4750 3400 4750
+$Comp
+L power:GNDD #PWR0106
+U 1 1 60E18502
+P 6000 5200
+F 0 "#PWR0106" H 6000 4950 50  0001 C CNN
+F 1 "GNDD" H 6004 5045 50  0000 C CNN
+F 2 "" H 6000 5200 50  0001 C CNN
+F 3 "" H 6000 5200 50  0001 C CNN
+	1    6000 5200
+	1    0    0    -1
+$EndComp
 $EndSCHEMATC
