File: KiCad/file591BC95F.sch (KiCad schematic (older format))
At the start: 54 parts, among them J203 V4, P201 Power Pole, P203 Power Pole, Q201 MUN5213DW1, Q202 DMP4025LSD, Q203 RJK0354DSP, U201 DAC081C085, U202 OPA171, U203 LTC3600, U204 MIC2196

Commit message: PCB Updates
Layout work
Parts:
- P201: symbol FlexFox80-rescue:CONN_01X02-ARDF-2-Band-MiniTx-rescue -> Connector_Generic:Conn_01x02
Changed lines of the file:
@@
 	2700 5450 2850 5450
 $Comp
-L FlexFox80-rescue:CONN_01X02-ARDF-2-Band-MiniTx-rescue P201
+L Connector_Generic:Conn_01x02 P201
 U 1 1 607F80D4
-P 6300 5100
-F 0 "P201" H 6300 5250 50  0000 C CNN
-F 1 "Power Pole" V 6450 5100 50  0000 C CNN
-F 2 "Oddities:Dummy_Empty_2" H 6300 5100 50  0001 C CNN
-F 3 "" H 6300 5100 50  0001 C CNN
-F 4 "2243-ASMPP30-1X2-RK-ND" H 6300 5100 50  0001 C CNN "Digi-Key Part No."
-F 5 "<a href=\"https://www.digikey.com/products/en?keywords=2243-ASMPP30-1X2-RK-ND\">Link</a>" H 6300 5100 60  0001 C CNN "Link"
-F 6 "TH" H 6300 5100 50  0001 C CNN "Manufacturer"
-F 7 "TH" H 6300 5100 50  0001 C CNN "Manufacturer PN"
-F 8 "TH" H 6300 5100 50  0001 C CNN "Description"
-	1    6300 5100
+P 6300 5050
+AR Path="/607F80D4" Ref="P201"  Part="1"
+AR Path="/591BC960/607F80D4" Ref="P201"  Part="1"
+F 0 "P201" H 6300 5200 50  0000 C CNN
+F 1 "Power Pole" V 6450 5050 50  0000 C CNN
+F 2 "Oddities:Dummy_Empty_2" H 6300 5050 50  0001 C CNN
+F 3 "" H 6300 5050 50  0001 C CNN
+F 4 "2243-ASMPP30-1X2-RK-ND" H 6300 5050 50  0001 C CNN "Digi-Key Part No."
+F 5 "<a href=\"https://www.digikey.com/products/en?keywords=2243-ASMPP30-1X2-RK-ND\">Link</a>" H 6300 5050 60  0001 C CNN "Link"
+F 6 "TH" H 6300 5050 50  0001 C CNN "Manufacturer"
+F 7 "TH" H 6300 5050 50  0001 C CNN "Manufacturer PN"
+F 8 "TH" H 6300 5050 50  0001 C CNN "Description"
+	1    6300 5050
 	-1   0    0    -1
 $EndComp

Commit message: AVR128DA48 Redesign
Kicad updates for new FlexFox design
Parts:
- removed C201, C203: 10uF, Capacitors_SMD:C_0805, symbol Device:C_Small
- removed L201: 10uH, Resistors_SMD:R_0805, symbol Device:INDUCTOR_SMALL
- removed U201: DAC081C085, Housings_SSOP:MSOP-8_3x3mm_Pitch0.65mm, symbol Analog_DAC:DAC081C085
- C202, C204, C206, C211, C212: LCSC Part Number (none) -> C360619
- C205, C216: LCSC Part Number (none) -> C84416
- C207: LCSC Part Number (none) -> C161109
- C208: LCSC Part Number (none) -> C344177
- C209, C215: LCSC Part Number (none) -> C444765
- C210: LCSC Part Number (none) -> C337455
- C213, C219: LCSC Part Number (none) -> C344171
- C214, C217: LCSC Part Number (none) -> C122333
- C218: LCSC Part Number (none) -> C527201
- D201, D202: LCSC Part Number (none) -> C110488
- L202, L203: footprint Inductors:CDR7D28MN -> Inductors:2020; Description FIXED IND 6.8UH 2.75A 46.3 MOHM -> FIXED IND 6.8UH 3A 39 MOHM SMD; Digi-Key Part No. 308-1328-1-ND -> 490-16286-1-ND; LCSC Part Number (none) -> C703749; Link <a href=\"https://www.digikey.com/products/en?keywords=308-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 -> <a href=\"https://www.digikey.com/products/en?keywords=490-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; Manufacturer Sumida America Components Inc. -> Murata Electronics; Manufacturer PN CDR7D28MNNP-6R8NC -> LQH5BPN6R8M38L
- Q201: LCSC Part Number (none) -> C95381
- Q202: LCSC Part Number (none) -> C150763
- Q203: LCSC Part Number (none) -> C919563
- R201, R205, R212: LCSC Part Number (none) -> C416820
- R202: LCSC Part Number (none) -> C218598
- R203, R208: LCSC Part Number (none) -> C139896
- R204: value 536k -> 392k; Description RES SMD 536K OHM 1% 1/8W 0805 -> RES SMD 392K OHM 1% 1/8W 0805; Digi-Key Part No. 311-536KCRCT-ND -> 311-392KCRCT-ND; LCSC Part Number (none) -> C273847; Link <a href=\"https://www.digikey.com/products/en?keywords=311-536KCRCT-ND\">Link</a> -> <a href=\"https://www.digikey.com/products/en?keywords=311-392KCRCT-ND\">Link</a>; Manufacturer PN RC0805FR-07536KL -> RC0805FR-07392KL
- R206: value 46.4k -> 27k; Description RES 46.4K OHM 1% 1/8W 0805 -> RES SMD 27K OHM 1% 1/8W 0805; Digi-Key Part No. RMCF0805FT46K4CT-ND -> 311-27.0KCRCT-ND; LCSC Part Number (none) -> C139896; Link <a href=\"https://www.digikey.com/products/en?keywords=RMCF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 -> <a href=\"https://www.digikey.com/products/en?keywords=311-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; Manufacturer Stackpole Electronics Inc -> Yageo; Manufacturer PN RMCF0805FT46K4 -> RC0805FR-0727KL
- R207, R209, R210: LCSC Part Number (none) -> C103905
- R211, R213, R214, R215, R216: LCSC Part Number (none) -> C38522
- R217: LCSC Part Number (none) -> C352257
- R218: LCSC Part Number (none) -> C728271
- U202: LCSC Part Number (none) -> C88036
- U203: LCSC Part Number (none) -> C580752
- U204: LCSC Part Number (none) -> C627808
Connections:
- net +3V3_L8: now also R204.1
- net DAC_OUTPUT: now reaches R203.2, W205.1
- no-connect marks 5 -> 3

Commit message: Gerber Updates
o Changed parts for C128, L203 and L204 to help with parts shortages
o Updated footprints
o Updated schematic
o Updated BOM
Parts:
- added JP201: Boost Bypass, Wire_Connections_Bridges:Solder-Jumper-NO-SMD-Pad_Small, symbol Device:Jumper_NO_Small
- L202, L203: footprint Inductors:2020 -> Inductors:CDR7D28MN; Description FIXED IND 6.8UH 3A 39 MOHM SMD -> FIXED IND 6.8UH 2.75A 46.3 MOHM; Digi-Key Part No. 490-16286-1-ND -> 308-1328-1-ND; LCSC Part Number C703749 -> (none); Link <a href=\"https://www.digikey.com/products/en?keywords=490-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 -> <a href=\"https://www.digikey.com/products/en?keywords=308-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; Manufacturer Murata Electronics -> Sumida America Components Inc.; Manufacturer PN LQH5BPN6R8M38L -> CDR7D28MNNP-6R8NC
Connections:
- wire segments 150 -> 155
Other:
- moved on the sheet: C202, C206, C209, C215, Q201A, Q202B, R201, R202, R209
