File: KiCad/FlexFox80.sch (KiCad schematic (older format))
At the start: 29 parts, among them J101 DIN-5_180degree, J102 Conn_01x02, Q102 IRF610, U101 TPS22810DBVT, U107 LM5134B

Commit message: Footprint Updates
Tweaks to PCB footprints.
Removed solder paste from unpopulated components
Parts:
- D102: footprint Diodes_SMD:SOD-123_Handsolder -> Diodes_SMD:SOD-123
Changed lines of the file:
@@
 U 1 1 628D7F12
 P 2600 2350
-F 0 "U101" H 2600 2717 50  0000 C CNN
-F 1 "TPS22810DBVT" H 2600 2626 50  0000 C CNN
+F 0 "U101" H 2600 2717 61  0000 C CNB
+F 1 "TPS22810DBVT" H 2600 2626 61  0000 C CNB
 F 2 "TO_SOT_Packages_SMD:SOT-23-6" H 2600 1650 50  0001 C CNN
 F 3 "http://www.ti.com/lit/ds/symlink/tps22810.pdf" H 2600 2350 50  0001 C CNN
@@
 F 0 "D102" H 3150 3050 50  0000 C CNN
 F 1 "4.7V" H 3150 2850 50  0000 C CNN
-F 2 "Diodes_SMD:SOD-123_Handsolder" H 3150 2950 50  0001 C CNN
+F 2 "Diodes_SMD:SOD-123" H 3150 2950 50  0001 C CNN
 F 3 "" H 3150 2950 50  0001 C CNN
 F 4 "BZT52C4V7-13FDICT-ND" H 3150 2950 50  0001 C CNN "Digi-Key Part No."

Commit message: Latest Gerbers
Gerbers with minor updates to silkscreen and D101, D301 footprints
Parts:
- D101: footprint TO_SOT_Packages_SMD:SOT-363-0.65 -> TO_SOT_Packages_SMD:SOT-363-0.65_MBD54
Changed lines of the file:
@@
 F 0 "D101" H 9150 2317 50  0000 C CNN
 F 1 "MBD54" H 9150 2226 50  0001 C CNN
-F 2 "TO_SOT_Packages_SMD:SOT-363-0.65" H 9150 2100 50  0001 C CNN
+F 2 "TO_SOT_Packages_SMD:SOT-363-0.65_MBD54" H 9150 2100 50  0001 C CNN
 F 3 "" H 9150 2100 50  0001 C CNN
 F 4 "MBD54DWT1GOSCT-ND" H 9150 2100 50  0001 C CNN "Digi-Key Part No."
